File: PCB/BamBam BoardController/BamBam BoardControllerS2.sch (KiCad schematic (older format))
At the start: 42 parts, among them IC1 CNY74-2, IC2 CNY74-2, P1 BremsOpto, Q1 IRLR2905z, Q2 IRLR2905z, Q3 IRLR2905z, Q4 IRLR2905z, Q5 IRLR2905z, X2 BLH, X3 AntiSpark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

Commit message: Auf BamBam angepasst. HC-05 Rahmen lag auf Pads BrmesOpto Text durch Bremse erstezt Gerber und Drill-Dateien generiert und gesichtet
Parts:
- P1: value BremsOpto -> Bremse
Changed lines of the file:
@@
 LIBS:contrib
 LIBS:valves
-LIBS:Teensy-cache
+LIBS:BamBam BoardController-cache
 EELAYER 25 0
 EELAYER END
@@
 P 4650 5800
 F 0 "P1" H 4650 6000 50  0000 C CNN
-F 1 "BremsOpto" H 4650 5600 50  0000 C CNN
+F 1 "Bremse" H 4650 5600 50  0000 C CNN
 F 2 "Pin_Headers:Pin_Header_Angled_1x03" H 4650 5800 60  0001 C CNN
 F 3 "" H 4650 5800 60  0000 C CNN

Commit message: Anpassung an die KiCAD Libs >02/2015 Einige kleine Korrekturen am Layout Anpassung der Mounting Holes mit NTPH (nicht durch kontaktieren) Zwei Texte im PCB zugefügt (Tx und Rx Ser2)
Other:
- moved on the sheet: R1, R10, R11, R12, R14, R16, R18, R2, R3, R4, R5, R6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
