File: PCB/BamBam BoardController/BamBam BoardController.kicad_pcb (KiCad board)
At the start: 2 copper layers, 85.1 x 52.3 mm, 74 parts, among them IC1 CNY74-2, IC2 CNY74-2, P1 Bremse, Q1 IRLR2905z, Q2 IRLR2905z, Q3 IRLR2905z, Q4 IRLR2905z, Q5 IRLR2905z, U1 TEENSY_3.1+4, U2 HC_05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

Commit message: Die Version 2.71 hat einige Veränderungen in den Bestückungstext bekommen, Verdeckte Texte wurden Verlagert und noch weitere Informationen an den Anschlüssen ergänzt. Eine Leiterbahn wurde im Querschnitt vergrößert und andere schöner verlegt.
Routing:
- net /A1: track 34.6 -> 36.1 mm
- net Net-(IC1-Pad5): track 65.9 -> 66.7 mm
- net /BamBam BoardController/Motor_Opto_A: track 16.2 -> 15.7 mm
- net Net-(R21-Pad2): track 5.80 -> 5.28 mm
Other:
- board text added: "3V3"
- board text added: "A1"
- board text added: "A10"
- board text added: "A11"
- board text added: "A14"
- board text added: "A3"
- board text added: "A7"
- board text added: "Data"
- board text added: "V 2.71 17.04.2015 Barney"
- board text removed: "V 2.7 31.03.2015 Barney"
